Commit message: first working Anymal_C hetergogeneous version - seems no NaNs in rewards

File: resources/robots/jackal/urdf/jackal.urdf (robot description, URDF)
Before this commit: robot jackal, 6 links, 5 joints
Links:
- link chassis_link: geometry collision box size=0.420 0.310 0.184; visual mesh filename=../meshes/jackal-base.stl scale=1 1 1
- link left_wheel_link: geometry collision cylinder length=0.040 radius=0.098; visual mesh filename=../meshes/jackal-wheel.stl scale=1 1 1
- link right_wheel_link: geometry collision cylinder length=0.040 radius=0.098; visual mesh filename=../meshes/jackal-wheel.stl scale=1 1 1
Joints:
- joint front_caster_joint: origin xyz=0.131 0 -0.02 rpy=0 0 0 -> xyz=0.131 0 0.02 rpy=0 0 0
- joint rear_caster_joint: origin xyz=-0.131 0 -0.02 rpy=0 0 0 -> xyz=-0.131 0 0.02 rpy=0 0 0
