Commit message: fixed anymal urdf for better collision with box

File: resources/robots/anymal_c/urdf/anymal_c.urdf (robot description, URDF)
Before this commit: robot anymal, 77 links, 76 joints
Links:
- link LF_HAA: geometry collision cylinder length=0.12 radius=0.055; visual mesh filename=../meshes/drive.dae scale=1.0 1.0 1.0
- link LF_HFE: geometry collision cylinder length=0.12 radius=0.055; visual mesh filename=../meshes/drive.dae scale=1.0 1.0 1.0
- link LF_hip_fixed: geometry collision box size=0.1 0.08 0.08; visual mesh filename=../meshes/hip_l.dae scale=1.0 1.0 1.0
- link LF_thigh_fixed: geometry collision box size=0.04 0.06 0.28; visual mesh filename=../meshes/thigh.dae scale=1.0 1.0 1.0
- link LH_HAA: geometry collision cylinder length=0.12 radius=0.055; visual mesh filename=../meshes/drive.dae scale=1.0 1.0 1.0
- link LH_HFE: geometry collision cylinder length=0.12 radius=0.055; visual mesh filename=../meshes/drive.dae scale=1.0 1.0 1.0
- link LH_hip_fixed: geometry collision box size=0.1 0.08 0.08; visual mesh filename=../meshes/hip_r.dae scale=1.0 1.0 1.0
- link LH_thigh_fixed: geometry collision box size=0.04 0.06 0.28; visual mesh filename=../meshes/thigh.dae scale=1.0 1.0 1.0
- link RF_HAA: geometry collision cylinder length=0.12 radius=0.055; visual mesh filename=../meshes/drive.dae scale=1.0 1.0 1.0
- link RF_HFE: geometry collision cylinder length=0.12 radius=0.055; visual mesh filename=../meshes/drive.dae scale=1.0 1.0 1.0
- link RF_hip_fixed: geometry collision box size=0.1 0.08 0.08; visual mesh filename=../meshes/hip_r.dae scale=1.0 1.0 1.0
- link RF_thigh_fixed: geometry collision box size=0.04 0.06 0.28; visual mesh filename=../meshes/thigh.dae scale=1.0 1.0 1.0
- link RH_HAA: geometry collision cylinder length=0.12 radius=0.055; visual mesh filename=../meshes/drive.dae scale=1.0 1.0 1.0
- link RH_HFE: geometry collision cylinder length=0.12 radius=0.055; visual mesh filename=../meshes/drive.dae scale=1.0 1.0 1.0
- link RH_hip_fixed: geometry collision box size=0.1 0.08 0.08; visual mesh filename=../meshes/hip_l.dae scale=1.0 1.0 1.0
- link RH_thigh_fixed: geometry collision box size=0.04 0.06 0.28; visual mesh filename=../meshes/thigh.dae scale=1.0 1.0 1.0
